Commit message: fix

File: urdf/AutoCar-Arm.xacro (robot description, xacro)
@@ -5,5 +5,5 @@
 <xacro:include filename="$(find auto_car_arm_description)/urdf/AutoCar-Arm.gazebo" />
 <xacro:include filename="$(find auto_car_arm_description)/urdf/open_manipulator_x.urdf.xacro" />
-<joint name="joint_arm" type="continuous">
+<joint name="joint_arm" type="fixed">
   <origin xyz="0.1525 0.0 0.246" rpy="0 0 0"/>
   <parent link="base_link"/>

Commit message: imu

File: urdf/AutoCar-Arm.xacro (robot description, xacro)
@@ -221,4 +221,22 @@
   <limit effort="10" lower="-0.34" upper="0.34" velocity="100"/>
 </joint>
+<link name="imu_link">
+  <collision>
+    <origin xyz="0 0 0" rpy="0 0 0"/>
+    <geometry>
+      <box size="0.1 0.1 0.1"/>
+    </geometry>
+  </collision>
+  <inertial>
+    <mass value="1e-5" />
+    <origin xyz="0 0 0" rpy="0 0 0"/>
+    <inertia ixx="1e-6" ixy="0" ixz="0" iyy="1e-6" iyz="0" izz="1e-6" />
+  </inertial>
+</link>
+<joint name="imu_joint" type="fixed">
+  <origin xyz="-0.039 0 0.0859" rpy="0 0 0"/>
+  <parent link="base_link"/>
+  <child link="imu_link"/>
+</joint>
 <joint name="joint_front_left" type="continuous">
   <origin xyz="0 0 0" rpy="0 0 0"/>
